Commit message: add checksum

File: config/gazebo_rArm.urdf (robot description, URDF)
Before this commit: robot rArm, 8 links, 7 joints
Joints:
- joint joint_2: limit lower=0 upper=1.57 effort=200 velocity=3 -> lower=-1.57 upper=1.57 effort=200 velocity=3
- joint joint_3: limit lower=0 upper=3.142 effort=200 velocity=3 -> lower=-0.52 upper=3.142 effort=200 velocity=3
- joint joint_4: limit lower=0 upper=3.142 effort=200 velocity=3 -> lower=-0.52 upper=3.142 effort=200 velocity=3
- joint joint_5: limit lower=0 upper=3.142 effort=200 velocity=3 -> lower=-0.52 upper=3.142 effort=200 velocity=3
- joint joint_6: limit lower=0 upper=3.142 effort=200 velocity=3 -> lower=-0.52 upper=3.142 effort=200 velocity=3
